File: Electronics/Controller/Controller.kicad_sch (KiCad schematic)
At the start: 0 parts

Commit message: PDF Update
Other:
- sheet Power+IO renamed Power and Output
- company: (none) -> findersee.fi
- title: (none) -> MQTT Output Controller
Changed lines of the file:
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@@
 (kicad_sch (version 20230121) (generator eeschema)
   (paper "A4")
+  (title_block
+    (title "MQTT Output Controller")
+    (date "2023-09-16")
+    (rev "1.0")
+    (company "findersee.fi")
+  )
   (wire (pts (xy 88.9 48.26) (xy 127 48.26))
     (stroke (width 0) (type default))
@@
     (stroke (width 0.3) (type solid) (color 194 0 0 1))
     (fill (color 132 132 132 1.0000))
-    (property "Sheetname" "Power+IO" (at 127 100.8884 0)
+    (property "Sheetname" "Power and Output" (at 127 100.8146 0)
       (effects (font (size 1.27 1.27)) (justify left bottom))
     )
-    (property "Sheetfile" "Pwr+IO.kicad_sch" (at 127 165.6846 0)
+    (property "Sheetfile" "Pwr+IO.kicad_sch" (at 127 165.7584 0)
       (effects (font (size 1.27 1.27)) (justify left top))
     )
@@
   )
   (sheet (at 44.45 38.1) (size 44.45 127) (fields_autoplaced)
-    (stroke (width 0.5) (type solid) (color 0 194 0 1))
-    (fill (color 255 255 255 1.0000))
+    (stroke (width 0.5) (type solid) (color 194 0 194 1))
+    (fill (color 255 153 0 1.0000))
     (property "Sheetname" "RP2040" (at 44.45 37.3884 0)
       (effects (font (size 1.27 1.27)) (justify left bottom))
