File: Electronics/Controller/Controller.kicad_pcb (KiCad board)
At the start: 4 copper layers, 82 x 29.4 mm, 87 parts, among them J201 SWD, J202 Expansion, J203 USB_B_Micro, J301 08B1-1X1T-06-F, J401 IO, Q401 AO3400A, Q402 AO3400A, Q403 AO3400A, SW201 BOOT, SW202 RESET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

Commit message: Manufacturing Commit
Parts:
- removed JP1: CLK JUMPER, Findersee_parts:0402_Jumper_3pin
- added R311: 0R, Resistor_SMD:R_0402_1005Metric, F.Cu at (107.0, 75.2)
- C308, C313: value 10n -> 10nF
- C403: value 100uF -> 68uF
- J201: footprint Connector_PinHeader_2.54mm:PinHeader_2x02_P2.54mm_Vertical -> Connector_PinHeader_2.54mm:PinHeader_1x03_P2.54mm_Vertical
- R310: value 12k4 -> 12.4k
- U203: value ASDMB-12.000MHZ-LC-T -> 12MHz; footprint Oscillator:Oscillator_SMD_Abracon_ASDMB-4Pin_2.5x2.0mm -> Oscillator:Oscillator_SMD_SeikoEpson_SG8002CE-4Pin_3.2x2.5mm
- U302: value ASDMB-25.000MHZ-LC-T -> 25 MHz; footprint Oscillator:Oscillator_SMD_Abracon_ASDMB-4Pin_2.5x2.0mm -> Oscillator:Oscillator_SMD_SeikoEpson_SG8002CE-4Pin_3.2x2.5mm
- moved J201 27.2 mm to (81.0, 62.5)
- moved C201 5.18 mm to (108.9, 67.0), turned to -90 degrees
- moved C315 3.04 mm to (108.6, 81.2), turned to 180 degrees
- moved U302 2.83 mm to (108.0, 78.5), turned to 90 degrees
- moved U203 1.36 mm to (105.9, 66.5), turned to 180 degrees
- moved F403 0.80 mm to (130.6, 72.6)
- moved C401 0.70 mm to (119.8, 66.0)
- moved C402 0.70 mm to (124.8, 66.7)
- moved C404 0.70 mm to (113.3, 65.1)
- moved C405 0.70 mm to (113.2, 63.5)
- moved D401 0.70 mm to (117.8, 68.2)
- moved D402 0.70 mm to (120.6, 62.5)
- moved FB401 0.70 mm to (124.1, 63.8)
- moved R401 0.70 mm to (116.5, 69.9)
- moved R402 0.70 mm to (114.6, 69.4)
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Connections:
- net /Power+IO/Boost renamed /Power and Output/Boost
- net /Power+IO/CH1 renamed /Power and Output/CH1
- net /Power+IO/CH2 renamed /Power and Output/CH2
- net /Power+IO/CH3 renamed /Power and Output/CH3
- net /Power+IO/SW renamed /Power and Output/SW
- U301 pad 30: Net-(JP1-C) -> Net-(U301-XI)
- U302 pad 3: Net-(JP1-B) -> Net-(U301-XI)
Routing:
- net Net-(J401-Pin_1): track 26.7 -> 0.00 mm
- net Net-(U301-XI): track 0.00 -> 8.44 mm
- net +3.3V: track 37.3 -> 44.6 mm, vias 19 -> 17
- net /Ethernet/ETH SCK: track 28.6 -> 24.3 mm
- net /Ethernet/ETH INT: track 29.3 -> 25.2 mm
- net Net-(JP1-B): track 3.82 -> 0.00 mm
- net Net-(JP1-C): track 3.68 -> 0.00 mm
- net /RP2040/SWCLK: track 24.2 -> 27.8 mm, vias 2 -> 1
- net /Ethernet/ETH RESET: track 23.5 -> 21.1 mm
- net Net-(U201-XIN): track 9.08 -> 7.12 mm
- net /Ethernet/Clock 25 MHz: track 33.1 -> 34.5 mm
- net /RP2040/RTC MISO: track 15.2 -> 16.5 mm
- net /RP2040/EXP SDA: track 17.4 -> 18.7 mm
- net /RP2040/USB+: track 26.5 -> 27.7 mm
- net /RP2040/USB-: track 26.5 -> 27.7 mm
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- added copper zone on In2.Cu, net +12V
- added copper zone on F.Cu, net Net-(J401-Pin_1)
- added copper zone on In2.Cu, net Net-(J401-Pin_1)
Other:
- board text added: "Findersee.fi 38/23"
- board text added: "SWD"
