File: Electronics/Controller/Controller.kicad_pcb (KiCad board)
At the start: 4 copper layers, 82 x 29.4 mm, 87 parts, among them J201 SWD, J202 Expansion, J203 USB_B_Micro, J301 08B1-1X1T-06-F, J401 IO, Q401 AO3400A, Q402 AO3400A, Q403 AO3400A, SW201 BOOT, SW202 RESET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

Commit message: Manufacturing commit 2
Parts:
- added D201: White, LED_SMD:LED_0603_1608Metric, F.Cu at (87.5, 63.9)
- added R203: 180, Resistor_SMD:R_0402_1005Metric, F.Cu at (85.2, 63.4)
- D403: footprint LED_SMD:LED_0805_2012Metric -> LED_SMD:LED_0603_1608Metric
Connections:
- U201 pad 39: unconnected-(U201-GPIO27-Pad39) -> Net-(D201-K)
Routing:
- net Net-(D201-K): track 0.00 -> 9.24 mm, vias 0 -> 2
- net /Ethernet/Clock 25 MHz: track 34.5 -> 30.4 mm
- net +3.3V: track 44.6 -> 46.2 mm
- net Net-(D201-A): track 0.00 -> 1.52 mm
- net /RP2040/SWCLK: track 27.8 -> 28.5 mm

Commit message: Pin goof fix
Parts:
- added D404: 1N5819, Diode_SMD:D_SOD-123, F.Cu at (71.6, 62.8)
- D402: value RBR5RSM40BTF -> 1N5819
- U202: value W25Q32JVSS -> IS25LP064
- moved J301 1.50 mm to (77.8, 79.5)
- moved R211 1.02 mm to (67.5, 62.4), turned to 180 degrees
- moved R212 0.73 mm to (68.6, 63.5), turned to 180 degrees
Connections:
- net Net-(J203-VBUS) renamed VBUS
- J202 pad 5: /RP2040/RTC MOSI -> /RP2040/RTC MISO
- J202 pad 9: /RP2040/RTC MISO -> /RP2040/RTC MOSI
- U201 pad 11: /RP2040/RTC MOSI -> /RP2040/RTC MISO
- U201 pad 14: /RP2040/RTC MISO -> /RP2040/RTC MOSI
- U201 pad 27: /Ethernet/ETH MOSI -> /Ethernet/ETH MISO
- U201 pad 30: /Ethernet/ETH MISO -> /Ethernet/ETH MOSI
Routing:
- net +12V: track 0.00 -> 62.1 mm, vias 8 -> 9
- net /Ethernet/ETH MISO: track 29.3 -> 20.5 mm
- net /Ethernet/ETH MOSI: track 19.9 -> 28.3 mm
- net VBUS: track 2.54 -> 9.21 mm
- net /RP2040/RTC MISO: track 16.5 -> 21.4 mm, vias 0 -> 1
- net /RP2040/RTC MOSI: track 21.5 -> 16.7 mm, vias 1 -> 0
- net Net-(U201-QSPI_SD3): track 12.5 -> 10.6 mm
- net Net-(U201-QSPI_SCLK): track 14.2 -> 12.4 mm
- net Net-(J301-TCT): track 14.8 -> 13.3 mm
- net /Ethernet/RX_P: track 8.29 -> 6.79 mm
- net /Ethernet/RX_N: track 8.29 -> 6.79 mm
- net /Ethernet/TX_P: track 9.04 -> 7.54 mm
- net /Ethernet/TX_N: track 9.00 -> 7.50 mm
- net Net-(J301-RCT): track 7.67 -> 6.21 mm
- net /RP2040/SWDIO: track 22.2 -> 21.5 mm
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
Commit message: Added library Fixed layout bugs Software improvements
Parts:
- C307: value 4.7uF -> 100nF
- H401, H402: footprint MountingHole:MountingHole_3.2mm_M3_DIN965 -> MountingHole:MountingHole_2.5mm
- R203, R409: value 180 -> 187R
- R301, R302, R303, R304: value 33 -> 33R2
- R305, R306, R308, R309: value 50 -> 48R7
- R310: value 12.4k -> 12k1
- moved C305 1.40 mm to (92.8, 85.2)
- moved C313 1.36 mm to (103.0, 87.0), turned to 0 degrees
- moved C304 1.01 mm to (102.0, 88.0), turned to 180 degrees
- moved R310 0.97 mm to (92.8, 83.8)
- moved C311 0.80 mm to (69.3, 69.8)
- moved J301 0.80 mm to (78.6, 79.5)
- moved C302 0.77 mm to (97.2, 87.8)
- moved C303 0.69 mm to (98.4, 87.8)
- moved C314 0.67 mm to (100.5, 87.5)
- moved R315 0.46 mm to (93.2, 77.4)
- moved R303 0.34 mm to (87.1, 83.6)
- moved C309 0.30 mm to (83.8, 83.6)
- moved C310 0.28 mm to (83.8, 82.5)
- moved C308 0.28 mm to (86.0, 85.7)
- moved R308 0.28 mm to (85.5, 82.0)
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Connections:
- net /RP2040/EXP SCL renamed /RP2040/EXP IO1
- net /RP2040/EXP SDA renamed /RP2040/EXP IO0
- C309 pad 1: /Ethernet/C_RX_P -> /Ethernet/C_RX_N
- C310 pad 1: /Ethernet/C_RX_N -> /Ethernet/C_RX_P
- J301 pad 4: /Ethernet/TX_N -> /Ethernet/TX_P
- J301 pad 5: /Ethernet/TX_P -> /Ethernet/TX_N
- R301 pad 1: /Ethernet/R_TX_P -> /Ethernet/R_TX_N
- R301 pad 2: /Ethernet/TX_P -> /Ethernet/TX_N
- R302 pad 1: /Ethernet/R_TX_N -> /Ethernet/R_TX_P
- R302 pad 2: /Ethernet/TX_N -> /Ethernet/TX_P
- R303 pad 1: /Ethernet/R_RX_P -> /Ethernet/R_RX_N
- R303 pad 2: /Ethernet/C_RX_P -> /Ethernet/C_RX_N
- R304 pad 1: /Ethernet/R_RX_N -> /Ethernet/R_RX_P
- R304 pad 2: /Ethernet/C_RX_N -> /Ethernet/C_RX_P
- R305 pad 1: /Ethernet/TX_P -> /Ethernet/TX_N
- R306 pad 1: /Ethernet/TX_N -> /Ethernet/TX_P
- R308 pad 2: /Ethernet/C_RX_N -> /Ethernet/C_RX_P
- R309 pad 2: /Ethernet/C_RX_P -> /Ethernet/C_RX_N
- U301 pad 1: /Ethernet/R_TX_P -> /Ethernet/R_TX_N
- U301 pad 2: /Ethernet/R_TX_N -> /Ethernet/R_TX_P
- U301 pad 5: /Ethernet/R_RX_N -> /Ethernet/R_RX_P
- U301 pad 6: /Ethernet/R_RX_P -> /Ethernet/R_RX_N
Routing:
- net +1V1: track 26.8 -> 22.6 mm, vias 4 -> 3
- net +3.3VA: track 15.4 -> 14.3 mm
- net /Ethernet/RX_N: track 6.79 -> 5.86 mm
- net /Ethernet/RX_P: track 6.79 -> 5.86 mm
- net Net-(J301-TCT): track 13.3 -> 12.4 mm
- net /Ethernet/TX_P: track 7.54 -> 6.74 mm
- net /Ethernet/TX_N: track 7.50 -> 6.74 mm
- net Net-(U301-TOCAP): track 2.30 -> 1.61 mm
- net Net-(U301-EXRES1): track 2.12 -> 2.79 mm
- net Net-(J301-RCT): track 6.21 -> 5.68 mm
- net +12V: track 62.1 -> 61.6 mm
- net GND: track 0.00 -> 0.02 mm, vias 72 -> 80
Other:
- board text added: "DIO GND CLK"

Commit message: Schematic and Layout update
Parts:
- removed C315: 100nF, Capacitor_SMD:C_0402_1005Metric
- removed FB401: 120R, Resistor_SMD:R_0805_2012Metric
- removed R311: 0R, Resistor_SMD:R_0402_1005Metric
- removed U302: 25 MHz, Oscillator:Oscillator_SMD_SeikoEpson_SG8002CE-4Pin_3.2x2.5mm
- added D405: 1N5819, Diode_SMD:D_SOD-123, F.Cu at (123.2, 63.3)
- D401: value 1N4148 -> 1N5819
- moved R211 3.79 mm to (71.2, 63.2)
- moved D404 3.61 mm to (68.2, 61.4), turned to 180 degrees
- moved R401 2.87 mm to (119.4, 69.9)
- moved R212 2.72 mm to (71.2, 64.3), turned to 0 degrees
- moved SW202 2.06 mm to (106.8, 62.9)
- moved C309 1.49 mm to (84.0, 82.1)
- moved R303 1.49 mm to (87.2, 82.1)
- moved C310 1.49 mm to (84.0, 81.0)
- moved R304 1.49 mm to (87.2, 81.0)
- moved R308 1.49 mm to (85.7, 80.5)
- moved R309 1.49 mm to (85.7, 82.6)
- moved C308 1.16 mm to (86.2, 84.6)
- moved L401 1.04 mm to (116.3, 63.9)
- moved C402 1.04 mm to (123.8, 66.5)
- moved C405 1.04 mm to (112.2, 63.2)
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Connections:
- U301 pad 30: Net-(U301-XI) -> /Ethernet/Clock 25 MHz
Routing:
- net Net-(U301-XI): track 8.44 -> 0.00 mm
- net /Ethernet/Clock 25 MHz: track 30.4 -> 37.8 mm
- net +3.3V: track 46.1 -> 41.5 mm
- net /RP2040/RST: track 11.4 -> 7.91 mm
- net +12V: track 61.6 -> 59.1 mm
- net +3.3VA: track 14.3 -> 16.0 mm
- net Net-(J301-TCT): track 12.4 -> 14.0 mm
- net /Ethernet/ETH MOSI: track 28.3 -> 27.2 mm
- net /Ethernet/ETH INT: track 25.2 -> 24.4 mm
- net /Ethernet/R_RX_N: track 9.08 -> 8.30 mm
- net /Ethernet/R_RX_P: track 9.08 -> 8.30 mm
- net VBUS: track 9.21 -> 8.46 mm
- net GND: vias 80 -> 81
Other:
- board text added: "Findersee.fi ${CURRENT_DATE}"
- board text removed: "Findersee.fi 38/23"

Commit message: Improvements
Parts:
- added C406: 10uF, Capacitor_SMD:C_0805_2012Metric, F.Cu at (123.8, 65.5)
- C404, C405: footprint Capacitor_SMD:C_0603_1608Metric -> Capacitor_SMD:C_0805_2012Metric
- D405: value 1N5819 -> SK36A-LTP; footprint Diode_SMD:D_SOD-123 -> Diode_SMD:D_SMA
- moved R411 8.26 mm to (121.2, 84.6)
- moved R410 7.92 mm to (120.7, 86.2)
- moved D405 6.28 mm to (129.5, 62.7)
- moved C402 3.99 mm to (121.8, 63.0), turned to 90 degrees
- moved C403 3.47 mm to (128.9, 68.3), turned to 0 degrees
- moved Q401 2.92 mm to (131.6, 78.6)
- moved Q402 2.92 mm to (131.6, 82.3)
- moved Q403 2.92 mm to (131.5, 85.9)
- moved R403 2.86 mm to (128.9, 78.2)
- moved R405 2.86 mm to (127.3, 77.6)
- moved R406 2.86 mm to (127.4, 81.3)
- moved R404 2.86 mm to (128.9, 81.8)
- moved F403 2.72 mm to (131.3, 75.2)
- moved R209 1.87 mm to (86.7, 67.3)
- moved R210 1.87 mm to (86.7, 66.3)
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Connections:
- C402 pad 1: Net-(D405-K) -> +12V
- D405 pad 1: Net-(D405-K) -> +12V
- D405 pad 2: +12V -> Net-(D405-A)
- J401 pad 7: +12V -> Net-(D405-A)
- U401 pad 4: Net-(D405-K) -> +12V
- U401 pad 5: Net-(D405-K) -> +12V
Routing:
- net Net-(Q403-G): track 2.87 -> 13.7 mm
- net +3.3V: track 41.5 -> 32.7 mm, vias 17 -> 18
- net VBUS: track 8.46 -> 0.00 mm
- net /Power and Output/CH2: track 37.7 -> 43.5 mm
- net /RP2040/USB-: track 27.7 -> 25.6 mm
- net /RP2040/USB+: track 27.7 -> 25.6 mm
- net /Power and Output/CH1: track 34.7 -> 36.7 mm
- net /RP2040/USB_RES_D-: track 3.28 -> 5.16 mm
- net /RP2040/USB_RES_D+: track 3.26 -> 5.08 mm
- net /Power and Output/CH3: track 37.1 -> 35.4 mm
- net /Ethernet/Clock 25 MHz: track 37.8 -> 36.9 mm
- net +3.3VA: track 16.0 -> 15.2 mm
- net Net-(J203-ID): track 2.25 -> 3.00 mm
- net Net-(D201-K): track 9.66 -> 10.2 mm
- net +12V: track 59.1 -> 58.8 mm, vias 9 -> 3
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- added copper zone on B.Cu, net Net-(D405-A)
- added copper zone on F.Cu, net Net-(D405-A)
- added copper zone on In1.Cu, net Net-(D405-A)
- added copper zone on In2.Cu, net Net-(D405-A)
- added copper zone on B.Cu, net Net-(J401-Pin_1)
- added copper zone on F.Cu, net VBUS
- removed copper zone on In2.Cu, net +12V
- removed copper zone on F.Cu, net Net-(D405-K)
- removed copper zone on F.Cu, net Net-(J401-Pin_1)
- removed copper zone on In2.Cu, net Net-(J401-Pin_1)
Other:
- board text added: "Findersee.fi ${CURRENT_DATE} Rev ${REVISION}"
- board text removed: "Findersee.fi ${CURRENT_DATE}"
