File: Electronics/Controller/Ethernet.kicad_sch (KiCad schematic)
At the start: 33 parts, among them J301 08B1-1X1T-06-F, U203 ASDMB-25.000MHZ-LC-T, U301 W5500

Commit message: PDF Update
Parts:
- C308, C313: value 10n -> 10nF
- R310: value 12k4 -> 12.4k
Other:
- company: (none) -> findersee.fi
- title: (none) -> MQTT Output Controller
Changed lines of the file:
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@@
 (kicad_sch (version 20230121) (generator eeschema)
   (paper "A3")
+  (title_block
+    (title "MQTT Output Controller")
+    (date "2023-09-16")
+    (rev "1.0")
+    (company "findersee.fi")
+  )
   (junction (at 88.9 63.5) (diameter 0) (color 0 0 0 0)
   )
@@
       (effects (font (size 1.27 1.27)))
     )
-    (property "Value" "10n" (at 185.42 113.03 90)
+    (property "Value" "10nF" (at 185.42 113.03 90)
       (effects (font (size 1 1)) (justify right))
     )
@@
   (symbol (lib_id "Device:C_Small") (at 226.06 82.55 90) (unit 1)
     (in_bom yes) (on_board yes) (dnp no) (fields_autoplaced)
-    (property "Reference" "C308" (at 226.0663 77.978 90)
-      (effects (font (size 1.27 1.27)))
-    )
-    (property "Value" "10n" (at 226.0663 79.899 90)
+    (property "Reference" "C308" (at 226.0663 76.8436 90)
+      (effects (font (size 1.27 1.27)))
+    )
+    (property "Value" "10nF" (at 226.0663 79.2678 90)
       (effects (font (size 1.27 1.27)))
     )
@@
       (effects (font (size 1.27 1.27)))
     )
-    (property "Value" "12k4" (at 177.8 110.49 90)
+    (property "Value" "12.4k" (at 177.8 110.49 90)
       (effects (font (size 0.8 0.8)))
     )

Commit message: Manufacturing Commit
Parts:
- removed JP1: CLK JUMPER, Findersee_parts:0402_Jumper_3pin, symbol Jumper:Jumper_3_Open
- added R311: 0R, Resistor_SMD:R_0402_1005Metric, symbol Device:R_Small
- U203: value ASDMB-25.000MHZ-LC-T -> 25 MHz; footprint Oscillator:Oscillator_SMD_Abracon_ASDMB-4Pin_2.5x2.0mm -> Oscillator:Oscillator_SMD_SeikoEpson_SG8002CE-4Pin_3.2x2.5mm; Manufacturer Abracon -> (none)
Connections:
- net Clock 25 MHz: now also R311.1
- net at U301.30 (XI): now also U203.3 (Out), R311.2
Changed lines of the file:
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@@
   (junction (at 78.74 63.5) (diameter 0) (color 0 0 0 0)
+  )
+  (junction (at 77.47 127) (diameter 0) (color 0 0 0 0)
   )
   (junction (at 213.36 58.42) (diameter 0) (color 0 0 0 0)
@@
     (stroke (width 0) (type default))
   )
+  (wire (pts (xy 77.47 137.16) (xy 77.47 127))
+    (stroke (width 0) (type default))
+  )
   (wire (pts (xy 189.23 123.19) (xy 189.23 125.73))
     (stroke (width 0) (type default))
@@
     (stroke (width 0) (type default))
   )
+  (wire (pts (xy 72.39 137.16) (xy 77.47 137.16))
+    (stroke (width 0) (type default))
+  )
   (wire (pts (xy 224.79 58.42) (xy 256.54 58.42))
     (stroke (width 0) (type default))
@@
     (stroke (width 0) (type default))
   )
-  (wire (pts (xy 78.74 127) (xy 78.74 121.92))
+  (wire (pts (xy 78.74 115.57) (xy 78.74 127))
     (stroke (width 0) (type default))
   )
@@
     (stroke (width 0) (type default))
   )
+  (wire (pts (xy 77.47 127) (xy 78.74 127))
+    (stroke (width 0) (type default))
+  )
   (wire (pts (xy 171.45 71.12) (xy 172.72 71.12))
     (stroke (width 0) (type default))
@@
     (stroke (width 0) (type default))
   )
-  (wire (pts (xy 76.2 109.22) (xy 78.74 109.22))
+  (wire (pts (xy 63.5 137.16) (xy 67.31 137.16))
     (stroke (width 0) (type default))
   )
@@
     (stroke (width 0) (type default))
   )
-  (wire (pts (xy 50.8 127) (xy 78.74 127))
+  (wire (pts (xy 50.8 127) (xy 77.47 127))
     (stroke (width 0) (type default))
   )
@@
     (stroke (width 0) (type default))
   )
-  (wire (pts (xy 82.55 115.57) (xy 100.33 115.57))
-    (stroke (width 0) (type default))
-  )
   (wire (pts (xy 171.45 110.49) (xy 175.26 110.49))
     (stroke (width 0) (type default))
@@
   )
   (wire (pts (xy 213.36 34.29) (xy 229.87 34.29))
+    (stroke (width 0) (type default))
+  )
+  (wire (pts (xy 78.74 115.57) (xy 100.33 115.57))
     (stroke (width 0) (type default))
   )
@@
     (effects (font (size 1.27 1.27)) (justify right))
   )
-  (hierarchical_label "Clock 25 MHz" (shape input) (at 76.2 109.22 180) (fields_autoplaced)
+  (hierarchical_label "Clock 25 MHz" (shape input) (at 63.5 137.16 180) (fields_autoplaced)
     (effects (font (size 1.27 1.27)) (justify right))
   )
@@
     )
   )
+  (symbol (lib_id "Device:R_Small") (at 69.85 137.16 90) (mirror x) (unit 1)
+    (in_bom no) (on_board yes) (dnp no)
+    (property "Reference" "R311" (at 69.8041 139.0246 90)
+      (effects (font (size 1.27 1.27)))
+    )
+    (property "Value" "0R" (at 69.85 137.16 90)
+      (effects (font (size 0.8 0.8)))
+    )
+    (property "Footprint" "Resistor_SMD:R_0402_1005Metric" (at 69.85 137.16 0)
+      (effects (font (size 1.27 1.27)) hide)
+    )
+    (property "Datasheet" "~" (at 69.85 137.16 0)
+      (effects (font (size 1.27 1.27)) hide)
+    )
+    (pin "1")
+    (pin "2")
+    (instances
+      (project "Controller"
+        (path "/a2ea94cb-4178-4727-9ac9-0e597b4a505d/5e10769e-2c76-442d-969e-a77f15adcbc3"
+          (reference "R311") (unit 1)
+        )
+      )
+    )
+  )
   (symbol (lib_id "power:+3.3V") (at 46.99 111.76 0) (unit 1)
     (in_bom yes) (on_board yes) (dnp no) (fields_autoplaced)
@@
       (effects (font (size 1.27 1.27)))
     )
-    (property "Value" "ASDMB-25.000MHZ-LC-T" (at 57.15 133.35 0)
-      (effects (font (size 1.27 1.27)))
-    )
-    (property "Footprint" "Oscillator:Oscillator_SMD_Abracon_ASDMB-4Pin_2.5x2.0mm" (at 40.64 127 0)
-      (effects (font (size 1.27 1.27)) hide)
-    )
-    (property "Datasheet" "https://abracon.com/Oscillators/ASDMB.pdf" (at 48.26 115.57 0)
-      (effects (font (size 1.27 1.27)) hide)
-    )
-    (property "Manufacturer" "Abracon" (at 40.64 127 0)
+    (property "Value" "25 MHz" (at 52.07 129.54 0)
+      (effects (font (size 1.27 1.27)))
+    )
+    (property "Footprint" "Oscillator:Oscillator_SMD_SeikoEpson_SG8002CE-4Pin_3.2x2.5mm" (at 40.64 127 0)
+      (effects (font (size 1.27 1.27)) hide)
+    )
+    (property "Datasheet" "" (at 48.26 115.57 0)
+      (effects (font (size 1.27 1.27)) hide)
+    )
+    (property "Manufacturer" "" (at 40.64 127 0)
       (effects (font (size 1.27 1.27)) hide)
     )
@@
         )
       )
-    )
-  )
-  (symbol (lib_id "Jumper:Jumper_3_Open") (at 78.74 115.57 90) (mirror x) (unit 1)
-    (in_bom yes) (on_board yes) (dnp no)
-    (property "Reference" "JP1" (at 76.6058 116.2137 90)
-      (effects (font (size 1.27 1.27)) (justify left))
-    )
-    (property "Value" "CLK JUMPER" (at 76.6058 114.2927 90)
-      (effects (font (size 1.27 1.27)) (justify left))
-    )
-    (property "Footprint" "Findersee_parts:0402_Jumper_3pin" (at 78.74 115.57 0)
-      (effects (font (size 1.27 1.27)) hide)
-    )
-    (property "Datasheet" "~" (at 78.74 115.57 0)
-      (effects (font (size 1.27 1.27)) hide)
-    )
-    (pin "1")
-    (pin "2")
-    (pin "3")
-    (instances
-      (project "Controller"
-        (path "/a2ea94cb-4178-4727-9ac9-0e597b4a505d/5e10769e-2c76-442d-969e-a77f15adcbc3"
-          (reference "JP1") (unit 1)
-        )
-      )

Commit message: Added library Fixed layout bugs Software improvements
Parts:
- C308, C313: symbol Device:C_Small -> Capacitors_0402:CAPC_10nF_X7R_25V_0402; Material (none) -> X7R; Voltage (none) -> 25V
- C309, C310: symbol Device:C_Small -> Capacitors_0402:CAPC_6.8nF_C0G_50V_0402; Material (none) -> C0G; Voltage (none) -> 50V
- C312: symbol Device:C_Small -> Capacitors_0402:CAPC_22nF_X7R_25V_0402; Material (none) -> X7R; Voltage (none) -> 25V
- C314: Package (none) -> 0402; Voltage (none) -> 6.3V
- C401: symbol Device:C_Small -> Capacitors_0402:CAPC_100nF_X5R_16V_0402; Material (none) -> X5R; Voltage (none) -> 16V
- C401: value 4.7uF -> 100nF; symbol Device:C_Small -> Capacitors_0402:CAPC_100nF_X5R_16V_0402; Material (none) -> X5R; Voltage (none) -> 16V
- R301, R302, R303, R304: value 33 -> 33R2; symbol Device:R_Small -> Resistors_0402:RESC_0402_33R2; Package (none) -> 0402
- R305, R306, R308, R309: value 50 -> 48R7; symbol Device:R_Small -> Resistors_0402:RESC_0402_48R7; Package (none) -> 0402
- R310: value 12.4k -> 12k1; symbol Device:R_Small -> Resistors_0402:RESC_0402_12k1; Package (none) -> 0402
- R311, R313, R314, R315: symbol Device:R_Small -> Resistors_0402:RESC_0402_0R; Package (none) -> 0402; now in the parts list
Connections:
- net C_RX_N: now also C309.1, R303.2, R309.2; no longer C310.1, R304.2, R308.2
- net C_RX_P: now also C310.1, R304.2, R308.2; no longer C309.1, R303.2, R309.2
- net R_RX_N: now also R303.1, U301.6 (RXP); no longer R304.1, U301.5 (RXN)
- net R_RX_P: now also R304.1, U301.5 (RXN); no longer R303.1, U301.6 (RXP)
- net R_TX_N: now also R301.1, U301.1 (TXN); no longer R302.1, U301.2 (TXP)
- net R_TX_P: now also R302.1, U301.2 (TXP); no longer R301.1, U301.1 (TXN)
- net TX_N: now also J301.5 (RD-), R301.2, R305.1; no longer J301.4 (RD+), R302.2, R306.1
- net TX_P: now also J301.4 (RD+), R302.2, R306.1; no longer J301.5 (RD-), R301.2, R305.1
Other:
- moved on the sheet: C309, C310, R301, R302, R303, R304

Commit message: Schematic and Layout update
Parts:
- removed C401: 100nF, Capacitor_SMD:C_0402_1005Metric, symbol Capacitors_0402:CAPC_100nF_X5R_16V_0402
- removed R311: 0R, Resistor_SMD:R_0402_1005Metric, symbol Resistors_0402:RESC_0402_0R
- removed U203: 25 MHz, Oscillator:Oscillator_SMD_SeikoEpson_SG8002CE-4Pin_3.2x2.5mm, symbol Oscillator:ASDMB-xxxMHz
- R313, R314, R315: now not fitted
Connections:
- net Clock 25 MHz: now also U301.30 (XI)
- no-connect marks 15 -> 14

Commit message: Improvements
Parts:
- renumbered C401 to C301, C401 to C302, C401 to C303, C401 to C304, C401 to C305, C401 to C306, C401 to C307
Changed lines of the file:
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@@
   (symbol (lib_id "Capacitors_0402:CAPC_100nF_X5R_16V_0402") (at 73.66 67.31 180) (unit 1)
     (in_bom yes) (on_board yes) (dnp no)
-    (property "Reference" "C401" (at 73.97 65.8862 0)
+    (property "Reference" "C304" (at 73.97 65.8862 0)
       (effects (font (size 0.8 0.8)) (justify right))
     )
@@
     (instances
       (project "Controller"
-        (path "/a2ea94cb-4178-4727-9ac9-0e597b4a505d/7516d84f-d298-4f48-8b5d-a736b2d19d1b"
-          (reference "C401") (unit 1)
-        )
-        (path "/a2ea94cb-4178-4727-9ac9-0e597b4a505d/b4def931-2d28-466e-81ae-3813755f1fa9"
-          (reference "C214") (unit 1)
-        )
         (path "/a2ea94cb-4178-4727-9ac9-0e597b4a505d/5e10769e-2c76-442d-969e-a77f15adcbc3"
           (reference "C304") (unit 1)
@@
   (symbol (lib_id "power:GND") (at 88.9 109.22 0) (unit 1)
     (in_bom yes) (on_board yes) (dnp no) (fields_autoplaced)
-    (property "Reference" "#PWR0213" (at 88.9 115.57 0)
+    (property "Reference" "#PWR0312" (at 88.9 115.57 0)
       (effects (font (size 1.27 1.27)) hide)
     )
@@
     (instances
       (project "Controller"
-        (path "/a2ea94cb-4178-4727-9ac9-0e597b4a505d/b4def931-2d28-466e-81ae-3813755f1fa9"
-          (reference "#PWR0213") (unit 1)
-        )
         (path "/a2ea94cb-4178-4727-9ac9-0e597b4a505d/5e10769e-2c76-442d-969e-a77f15adcbc3"
           (reference "#PWR0312") (unit 1)
@@
   (symbol (lib_id "power:PWR_FLAG") (at 304.8 45.72 0) (unit 1)
     (in_bom yes) (on_board yes) (dnp no) (fields_autoplaced)
-    (property "Reference" "#FLG0402" (at 304.8 43.815 0)
+    (property "Reference" "#FLG0301" (at 304.8 43.815 0)
       (effects (font (size 1.27 1.27)) hide)
     )
@@
     (instances
       (project "Controller"
-        (path "/a2ea94cb-4178-4727-9ac9-0e597b4a505d/7516d84f-d298-4f48-8b5d-a736b2d19d1b"
-          (reference "#FLG0402") (unit 1)
-        )
         (path "/a2ea94cb-4178-4727-9ac9-0e597b4a505d/5e10769e-2c76-442d-969e-a77f15adcbc3"
           (reference "#FLG0301") (unit 1)
@@
   (symbol (lib_id "Capacitors_0402:CAPC_100nF_X5R_16V_0402") (at 68.58 67.31 180) (unit 1)
     (in_bom yes) (on_board yes) (dnp no)
-    (property "Reference" "C401" (at 68.89 65.8862 0)
+    (property "Reference" "C303" (at 68.89 65.8862 0)
       (effects (font (size 0.8 0.8)) (justify right))
     )
@@
     (instances
       (project "Controller"
-        (path "/a2ea94cb-4178-4727-9ac9-0e597b4a505d/7516d84f-d298-4f48-8b5d-a736b2d19d1b"
-          (reference "C401") (unit 1)
-        )
-        (path "/a2ea94cb-4178-4727-9ac9-0e597b4a505d/b4def931-2d28-466e-81ae-3813755f1fa9"
-          (reference "C214") (unit 1)
-        )
         (path "/a2ea94cb-4178-4727-9ac9-0e597b4a505d/5e10769e-2c76-442d-969e-a77f15adcbc3"
           (reference "C303") (unit 1)
@@
   (symbol (lib_id "Capacitors_0402:CAPC_100nF_X5R_16V_0402") (at 78.74 67.31 180) (unit 1)
     (in_bom yes) (on_board yes) (dnp no)
-    (property "Reference" "C401" (at 79.05 65.8862 0)
+    (property "Reference" "C305" (at 79.05 65.8862 0)
       (effects (font (size 0.8 0.8)) (justify right))
     )
@@
     (instances
       (project "Controller"
-        (path "/a2ea94cb-4178-4727-9ac9-0e597b4a505d/7516d84f-d298-4f48-8b5d-a736b2d19d1b"
-          (reference "C401") (unit 1)
-        )
-        (path "/a2ea94cb-4178-4727-9ac9-0e597b4a505d/b4def931-2d28-466e-81ae-3813755f1fa9"
-          (reference "C214") (unit 1)
-        )
         (path "/a2ea94cb-4178-4727-9ac9-0e597b4a505d/5e10769e-2c76-442d-969e-a77f15adcbc3"
           (reference "C305") (unit 1)
@@
   (symbol (lib_id "Capacitors_0402:CAPC_100nF_X5R_16V_0402") (at 83.82 67.31 180) (unit 1)
     (in_bom yes) (on_board yes) (dnp no)
-    (property "Reference" "C401" (at 84.13 65.8862 0)
+    (property "Reference" "C306" (at 84.13 65.8862 0)
       (effects (font (size 0.8 0.8)) (justify right))
     )
@@
     (instances
       (project "Controller"
-        (path "/a2ea94cb-4178-4727-9ac9-0e597b4a505d/7516d84f-d298-4f48-8b5d-a736b2d19d1b"
-          (reference "C401") (unit 1)
-        )
-        (path "/a2ea94cb-4178-4727-9ac9-0e597b4a505d/b4def931-2d28-466e-81ae-3813755f1fa9"
-          (reference "C214") (unit 1)
-        )
         (path "/a2ea94cb-4178-4727-9ac9-0e597b4a505d/5e10769e-2c76-442d-969e-a77f15adcbc3"
           (reference "C306") (unit 1)
@@
   (symbol (lib_id "Capacitors_0402:CAPC_100nF_X5R_16V_0402") (at 63.5 67.31 180) (unit 1)
     (in_bom yes) (on_board yes) (dnp no)
-    (property "Reference" "C401" (at 63.81 65.8862 0)
+    (property "Reference" "C302" (at 63.81 65.8862 0)
       (effects (font (size 0.8 0.8)) (justify right))
     )
@@
     (instances
       (project "Controller"
-        (path "/a2ea94cb-4178-4727-9ac9-0e597b4a505d/7516d84f-d298-4f48-8b5d-a736b2d19d1b"
-          (reference "C401") (unit 1)
-        )
-        (path "/a2ea94cb-4178-4727-9ac9-0e597b4a505d/b4def931-2d28-466e-81ae-3813755f1fa9"
-          (reference "C214") (unit 1)
-        )
         (path "/a2ea94cb-4178-4727-9ac9-0e597b4a505d/5e10769e-2c76-442d-969e-a77f15adcbc3"
           (reference "C302") (unit 1)
@@
   (symbol (lib_id "Capacitors_0402:CAPC_100nF_X5R_16V_0402") (at 88.9 67.31 180) (unit 1)
     (in_bom yes) (on_board yes) (dnp no)
-    (property "Reference" "C401" (at 89.21 65.8862 0)
+    (property "Reference" "C307" (at 89.21 65.8862 0)
       (effects (font (size 0.8 0.8)) (justify right))
     )
@@
     (instances
       (project "Controller"
-        (path "/a2ea94cb-4178-4727-9ac9-0e597b4a505d/7516d84f-d298-4f48-8b5d-a736b2d19d1b"
-          (reference "C401") (unit 1)
-        )
-        (path "/a2ea94cb-4178-4727-9ac9-0e597b4a505d/b4def931-2d28-466e-81ae-3813755f1fa9"
-          (reference "C214") (unit 1)
-        )
         (path "/a2ea94cb-4178-4727-9ac9-0e597b4a505d/5e10769e-2c76-442d-969e-a77f15adcbc3"
           (reference "C307") (unit 1)
@@
   (symbol (lib_id "Capacitors_0402:CAPC_100nF_X5R_16V_0402") (at 58.42 67.31 180) (unit 1)
     (in_bom yes) (on_board yes) (dnp no)
-    (property "Reference" "C401" (at 58.73 65.8862 0)
+    (property "Reference" "C301" (at 58.73 65.8862 0)
       (effects (font (size 0.8 0.8)) (justify right))
     )
@@
     (instances
       (project "Controller"
-        (path "/a2ea94cb-4178-4727-9ac9-0e597b4a505d/7516d84f-d298-4f48-8b5d-a736b2d19d1b"
-          (reference "C401") (unit 1)
-        )
-        (path "/a2ea94cb-4178-4727-9ac9-0e597b4a505d/b4def931-2d28-466e-81ae-3813755f1fa9"
-          (reference "C214") (unit 1)
-        )
         (path "/a2ea94cb-4178-4727-9ac9-0e597b4a505d/5e10769e-2c76-442d-969e-a77f15adcbc3"
           (reference "C301") (unit 1)
