File: Electronics/RTC_Module/RTC_Module.kicad_pcb (KiCad board)
At the start: 2 copper layers, 32.4 x 36.6 mm, 21 parts, among them J101 EXT_UART, J102 Expansion, J103 EXP I^{2}C, U101 DS3234S, U102 DS1307ZN+, Y101 32.768k

Commit message: Manufacturing Commit
Other:
- board text added: "Findersee.fi 38/23"
Changed lines of the file:
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@@
     (property "ki_keywords" "R resistor")
     (attr smd exclude_from_bom)
-    (fp_text reference "R106" (at -2.35 -0.15) (layer "F.SilkS")
+    (fp_text reference "R106" (at 0.04 1.1) (layer "F.SilkS")
         (effects (font (size 0.6 0.6) (thickness 0.15)))
     )
@@
   (gr_rect (start 70 103.5) (end 102.4 140.1)
     (stroke (width 0.1) (type default)) (fill none) (layer "Edge.Cuts"))
+  (gr_text "Findersee.fi\n38/23" (at 73.2 109.9 90) (layer "B.SilkS")
+    (effects (font (size 1 1) (thickness 0.15)) (justify left bottom mirror))
+  )
   (dimension (type aligned) (layer "Cmts.User")
     (pts (xy 102.4 140.1) (xy 70 140.1))
