File: Electronics/RTC_Module/RTC_Module.kicad_pcb (KiCad board)
At the start: 2 copper layers, 32.4 x 36.6 mm, 21 parts, among them J101 EXT_UART, J102 Expansion, J103 EXP I^{2}C, U101 DS3234S, U102 DS1307ZN+, Y101 32.768k

Commit message: Pin goof fix
Connections:
- J102 pad 5: /RTC MOSI -> /RTC MISO
- J102 pad 9: /RTC MISO -> /RTC MOSI
Routing:
- net /RTC SCK: track 15.6 -> 10.5 mm
- net /RTC ~{CS}: track 15.2 -> 17.9 mm
- net /RX: track 43.2 -> 45.5 mm
- net /LED2: track 47.6 -> 49.7 mm
- net /TX: track 39.2 -> 40.5 mm
- net /RTC MISO: track 28.7 -> 28.3 mm, vias 0 -> 2

Commit message: Added library Fixed layout bugs Software improvements
Parts:
- D101: value RBR5RSM40BTF -> 1N5819
Connections:
- net /EXP SCL renamed /IO 2
- J102 pad 10: /EXP SDA -> /IO 1
- J103 pad 2: /EXP SDA -> /IO 1
- R108 pad 1: /EXP SDA -> /IO 1
- U101 pad 5: unconnected-(U101-~{INT}-Pad5) -> /IO 1
Routing:
- net /IO 1: track 0.00 -> 12.3 mm, vias 0 -> 1
- net /EXP SDA: track 10.8 -> 0.00 mm
