File: Electronics/RTC_Module/RTC_Module.kicad_sch (KiCad schematic)
At the start: 21 parts, among them J101 EXT_UART, J103 EXP I^{2}C, J202 Expansion, U204 DS3234S, U205 DS1307ZN+, Y201 32.768k

Commit message: Pin goof fix
Connections:
- net RTC MISO: now also J202.5 (Pin_5); no longer J202.9 (Pin_9)
- net RTC MOSI: now also J202.9 (Pin_9); no longer J202.5 (Pin_5)
Changed lines of the file:
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@@
     (effects (font (size 1.27 1.27)) (justify left bottom))
   )
-  (label "RTC MISO" (at 73.66 86.36 180) (fields_autoplaced)
+  (label "RTC MISO" (at 73.66 76.2 180) (fields_autoplaced)
     (effects (font (size 1.27 1.27)) (justify right bottom))
   )
@@
     (effects (font (size 1.27 1.27)) (justify left bottom))
   )
-  (label "RTC MOSI" (at 73.66 76.2 180) (fields_autoplaced)
+  (label "RTC MOSI" (at 73.66 86.36 180) (fields_autoplaced)
     (effects (font (size 1.27 1.27)) (justify right bottom))
   )

Commit message: DS3234_Driver Fixes Added watch dog reset
Connections:
- net EXP SCL: now also U204.5 (~{INT})
- no-connect marks 5 -> 4
Changed lines of the file:
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@@
   (no_connect (at 191.77 73.66))
   (no_connect (at 220.98 38.1))
-  (no_connect (at 220.98 43.18))
   (no_connect (at 219.71 129.54))
   (no_connect (at 191.77 62.23))
@@
     (stroke (width 0) (type default))
   )
+  (wire (pts (xy 220.98 43.18) (xy 223.52 43.18))
+    (stroke (width 0) (type default))
+  )
   (wire (pts (xy 68.58 62.23) (xy 68.58 66.04))
     (stroke (width 0) (type default))
@@
     (effects (font (size 1.27 1.27)) (justify left bottom))
   )
+  (label "EXP SCL" (at 223.52 43.18 0) (fields_autoplaced)
+    (effects (font (size 1.27 1.27)) (justify left bottom))
+  )

Commit message: Added library Fixed layout bugs Software improvements
Parts:
- D404: value RBR5RSM40BTF -> 1N5819
Connections:
- net EXP SCL renamed IO 2
- net IO 2: no longer U204.5 (~{INT})
- net EXP SDA renamed IO 1
- net IO 1: now also U204.5 (~{INT})
Changed lines of the file:
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@@
     (effects (font (size 1.27 1.27)) (justify left bottom))
   )
-  (label "EXP SDA" (at 73.66 88.9 180) (fields_autoplaced)
+  (label "IO 1" (at 73.66 88.9 180) (fields_autoplaced)
     (effects (font (size 1.27 1.27)) (justify right bottom))
   )
@@
     (effects (font (size 1.27 1.27)) (justify left bottom))
   )
-  (label "EXP SCL" (at 223.52 43.18 0) (fields_autoplaced)
+  (label "IO 1" (at 223.52 43.18 0) (fields_autoplaced)
     (effects (font (size 1.27 1.27)) (justify left bottom))
   )
@@
     (effects (font (size 1.27 1.27)) (justify right bottom))
   )
-  (label "EXP SCL" (at 73.66 91.44 180) (fields_autoplaced)
+  (label "IO 2" (at 73.66 91.44 180) (fields_autoplaced)
     (effects (font (size 1.27 1.27)) (justify right bottom))
   )
@@
       (effects (font (size 1.27 1.27)) (justify right))
     )
-    (property "Value" " RBR5RSM40BTF" (at 164.592 33.2813 90)
+    (property "Value" "1N5819" (at 164.592 33.2813 90)
       (effects (font (size 1.27 1.27)) (justify right))
     )
